File: hardware/motor_board/02_control.kicad_sch (KiCad schematic)
At the start: 30 parts, among them U7 RP2350A, U8 W25Q128JVUXIQ, U9 SPX3819M5-3.3, Y1 12MHz

Commit message: Every placed part gets an LCSC number; 3D inductors and part colours fixed
LCSC (hardware/parts/lcsc.csv, 76 rows): every part the assembler places on
boards A (120) and S (173) now has a number, joined into the 3D part pane.
Chosen from the sister board's BOM where it had the part, JLC basic parts
where the rating allowed, each matched to the net it sits on and checked
against JLCPCB's library (model, package, rating, stock) on 2026-09-24. The
notes say why where it was not obvious: 100 V X7R/C0G on VBUS, 0.1% thin
film for the dividers, a Vishay WSL metal-strip jumper for phase C's 0R
(75 A, where a thick-film 0R carries a few), a CL 20 pF crystal for the
27 pF caps, the RGB LED placed rotated 180 deg. export_3d.py warns about any
placed part without a number; copper features (lands, lead pads, bosses)
get no LCSC row in the pane.

Two values changed because nothing stocked matches them:
- Shunts 1m6 -> 2m0 (WSLP20102L000FEA): no 1.6 mOhm 2010 exists at LCSC or
  JLCPCB. The pair is 1.0 mOhm, 50 mV/A, +-29.0 A worst case -- 2.5% over
  the 28.3 A peak, the margin draft 0.3 turned down, taken knowingly.
  geometry.SHUNT_EACH follows; spec, README and status page re-derive the
  sense chain and the loss budget (10.72 W, <= 6.67 K/W, >= 100 cm2).
- Flash W25Q128 -> W25Q16JVUXIQ: no 128 Mbit part comes in USON 2x3; this
  is the RP2350 reference design's part. Derived symbol renamed W25Q16JV.
Schematics regenerated in a scratch copy and only the changed sheets copied
back (diffed: nothing else moved); the routed boards' value fields patched
in place. ERC 0 and DRC 0 on both; KiCad's parity list is HEAD's minus one
(board A's U8 value mismatch). Board S's plan drawings and parts table
regenerated, which also brings them back in line with the final placement.

3D export:
- Board S's two buck inductors were invisible: kicad-cli 9.0.8 meshes a STEP
  that is an assembly of sub-assemblies (KiCad's own SWPA4030S) as empty
  nodes, silently. tools/flatten_step.py flattens it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
Parts:
- U8: value W25Q128JVUXIQ -> W25Q16JVUXIQ; symbol servodrive:W25Q128JV -> servodrive:W25Q16JV
Changed lines of the file:
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@@
 )
 	(symbol
-		(lib_id "servodrive:W25Q128JV")
+		(lib_id "servodrive:W25Q16JV")
 		(at 38.1000 355.6000 0)
 		(unit 1)
@@
 			(at 27.9400 340.3600 0)
 			(effects (font (size 1.27 1.27)) (justify left)))
-		(property "Value" "W25Q128JVUXIQ"
+		(property "Value" "W25Q16JVUXIQ"
 			(at 27.9400 370.8400 0)
 			(effects (font (size 1.27 1.27)) (justify left)))
