File: hardware/single_board/01_power_stage.kicad_sch (KiCad schematic)
At the start: 76 parts, among them Q1 BSC030N08NS5, Q2 BSC030N08NS5, Q3 BSC030N08NS5, Q4 BSC030N08NS5, Q5 BSC030N08NS5, Q6 BSC030N08NS5, U1 EG2103, U2 EG2103, U3 EG2103, U4 INA241A3, U5 INA241A3, U6 INA241A3

Commit message: Every placed part gets an LCSC number; 3D inductors and part colours fixed
LCSC (hardware/parts/lcsc.csv, 76 rows): every part the assembler places on
boards A (120) and S (173) now has a number, joined into the 3D part pane.
Chosen from the sister board's BOM where it had the part, JLC basic parts
where the rating allowed, each matched to the net it sits on and checked
against JLCPCB's library (model, package, rating, stock) on 2026-09-24. The
notes say why where it was not obvious: 100 V X7R/C0G on VBUS, 0.1% thin
film for the dividers, a Vishay WSL metal-strip jumper for phase C's 0R
(75 A, where a thick-film 0R carries a few), a CL 20 pF crystal for the
27 pF caps, the RGB LED placed rotated 180 deg. export_3d.py warns about any
placed part without a number; copper features (lands, lead pads, bosses)
get no LCSC row in the pane.

Two values changed because nothing stocked matches them:
- Shunts 1m6 -> 2m0 (WSLP20102L000FEA): no 1.6 mOhm 2010 exists at LCSC or
  JLCPCB. The pair is 1.0 mOhm, 50 mV/A, +-29.0 A worst case -- 2.5% over
  the 28.3 A peak, the margin draft 0.3 turned down, taken knowingly.
  geometry.SHUNT_EACH follows; spec, README and status page re-derive the
  sense chain and the loss budget (10.72 W, <= 6.67 K/W, >= 100 cm2).
- Flash W25Q128 -> W25Q16JVUXIQ: no 128 Mbit part comes in USON 2x3; this
  is the RP2350 reference design's part. Derived symbol renamed W25Q16JV.
Schematics regenerated in a scratch copy and only the changed sheets copied
back (diffed: nothing else moved); the routed boards' value fields patched
in place. ERC 0 and DRC 0 on both; KiCad's parity list is HEAD's minus one
(board A's U8 value mismatch). Board S's plan drawings and parts table
regenerated, which also brings them back in line with the final placement.

3D export:
- Board S's two buck inductors were invisible: kicad-cli 9.0.8 meshes a STEP
  that is an assembly of sub-assemblies (KiCad's own SWPA4030S) as empty
  nodes, silently. tools/flatten_step.py flattens it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
Parts:
- R105, R106, R205, R206: value 1m6 -> 2m0
Changed lines of the file:
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@@
 			(at 28.1940 158.7500 0)
 			(effects (font (size 1.27 1.27)) (justify left)))
-		(property "Value" "1m6"
+		(property "Value" "2m0"
 			(at 28.1940 171.4500 0)
 			(effects (font (size 1.27 1.27)) (justify left)))
@@
 			(at 57.4040 158.7500 0)
 			(effects (font (size 1.27 1.27)) (justify left)))
-		(property "Value" "1m6"
+		(property "Value" "2m0"
 			(at 57.4040 171.4500 0)
 			(effects (font (size 1.27 1.27)) (justify left)))
@@
 			(at 28.1940 364.4900 0)
 			(effects (font (size 1.27 1.27)) (justify left)))
-		(property "Value" "1m6"
+		(property "Value" "2m0"
 			(at 28.1940 377.1900 0)
 			(effects (font (size 1.27 1.27)) (justify left)))
@@
 			(at 57.4040 364.4900 0)
 			(effects (font (size 1.27 1.27)) (justify left)))
-		(property "Value" "1m6"
+		(property "Value" "2m0"
 			(at 57.4040 377.1900 0)
 			(effects (font (size 1.27 1.27)) (justify left)))

Commit message: Board S schematic: drawn as a person would draw it, and on the page
The sheets were a grid of parts with a stub and a label on every pin.
tools/schdraw.py now draws a netlist from a hand-written layout: parts
placed and turned, wires between the pins that belong together, T-joins
split with a junction dot, ground and supply symbols on power pins, labels
only where a signal leaves its block. tools/schlayout_s.py is board S's
five sheets: signal left to right, supplies up, ground down, each part's
support parts at the pin they serve, dashed frames and notes. The header
pins and the notes follow the netlist, so a pin-map change redraws itself.

The drawing cannot change the circuit: every sheet is checked against
schematic_s's netlist before it is written, and `schdraw.py --check s`
compares KiCad's own netlist export net by net. It matches; ERC is 0 at
every severity; PCB parity is unchanged (the same 219 reports as before).

Found on the way: a symbol's instance path must be /<root>/<sheet>. With
the root left out, as schematic.py writes it, KiCad joins labelled nets
but silently drops every net that is only wire -- the old sheets labelled
every pin, so it never showed. Board A's generator is unchanged.

single.html: an SCH tab in the viewer (sch.js) -- the sheets as KiCad
plots them, a sheet list, drag to pan, scroll to zoom, a PDF of the lot.
tools/regen.py plots them into img/sch/s/ (--sch for that alone).

Co-Authored-By: Claude Opus 5.5 (1M context) <noreply@anthropic.com>
Connections:
- net GH_A: no longer names the net of Q1.4 (G), R101.2, R109.1
- net GH_B: no longer names the net of Q3.4 (G), R201.2, R209.1
- net GH_C: no longer names the net of Q5.4 (G), R301.2, R309.1
- net GL_A: no longer names the net of Q2.4 (G), R102.2, R110.1
- net GL_B: no longer names the net of Q4.4 (G), R202.2, R210.1
- net GL_C: no longer names the net of Q6.4 (G), R302.2, R310.1
- net HO_A: no longer names the net of R101.1, U1.7 (HO)
- net HO_B: no longer names the net of R201.1, U2.7 (HO)
- net HO_C: no longer names the net of R301.1, U3.7 (HO)
- net LO_A: no longer names the net of R102.1, U1.5 (LO)
- net LO_B: no longer names the net of R202.1, U2.5 (LO)
- net LO_C: no longer names the net of R302.1, U3.5 (LO)
- net SNSN_A: no longer names the net of C108.2, R108.2, U4.1 (-)
- net SNSN_B: no longer names the net of C208.2, R208.2, U5.1 (-)
- net SNSN_C: no longer names the net of C308.2, R308.2, U6.1 (-)
- net SNSP_A: no longer names the net of C108.1, R107.1, U4.8 (+)
- net SNSP_B: no longer names the net of C208.1, R207.1, U5.8 (+)
- net SNSP_C: no longer names the net of C308.1, R307.1, U6.8 (+)
- net SNUB_A: no longer names the net of C109.2, R113.1
- net SNUB_B: no longer names the net of C209.2, R213.1
- net SNUB_C: no longer names the net of C309.2, R313.1
- net VB_A: no longer names the net of C105.1, D101.1 (K), U1.8 (VB)
- net VB_B: no longer names the net of C205.1, D201.1 (K), U2.8 (VB)
- net VB_C: no longer names the net of C305.1, D301.1 (K), U3.8 (VB)
Other:
- note added: "Each phase is an EG2103 half-bridge driver on a pair of BSC030N08NS5: bootstrap diode and capacitor (D101, C105 on phase A), 2R2 gate resistors, 10k gate-source pull-downs. HIN and LIN are held low (R111, R112): with both low the EG2103 turns the low side on, so a CPU in reset brakes the motor. Inline shunt: two 2m0 in parallel between the switch node and the motor lead, Kelvin-sensed through 10R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"
- note added: "Notes"
- note added: "Phase A"
- note added: "Phase B"
- note added: "Phase C"
- note removed: "phase A: FET temperature"
- note removed: "phase A: gate drive"
- note removed: "phase A: half bridge"
- note removed: "phase A: phase output and sense"
- note removed: "phase A: snubber"
- note removed: "phase B: gate drive"
- note removed: "phase B: half bridge"
- note removed: "phase B: phase output and sense"
- note removed: "phase B: snubber"
- note removed: "phase C: gate drive"
- note removed: "phase C: half bridge"
- note removed: "phase C: phase output and sense"
- note removed: "phase C: snubber"
- moved on the sheet: C101, C102, C103, C104, C105, C106, C108, C109, C201, C202, C203, C204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
