File: hardware/single_board/02_control.kicad_sch (KiCad schematic)
At the start: 30 parts, among them U7 RP2350A, U8 W25Q16JVUXIQ, U9 SPX3819M5-3.3, Y1 12MHz

Commit message: Board S schematic: drawn as a person would draw it, and on the page
The sheets were a grid of parts with a stub and a label on every pin.
tools/schdraw.py now draws a netlist from a hand-written layout: parts
placed and turned, wires between the pins that belong together, T-joins
split with a junction dot, ground and supply symbols on power pins, labels
only where a signal leaves its block. tools/schlayout_s.py is board S's
five sheets: signal left to right, supplies up, ground down, each part's
support parts at the pin they serve, dashed frames and notes. The header
pins and the notes follow the netlist, so a pin-map change redraws itself.

The drawing cannot change the circuit: every sheet is checked against
schematic_s's netlist before it is written, and `schdraw.py --check s`
compares KiCad's own netlist export net by net. It matches; ERC is 0 at
every severity; PCB parity is unchanged (the same 219 reports as before).

Found on the way: a symbol's instance path must be /<root>/<sheet>. With
the root left out, as schematic.py writes it, KiCad joins labelled nets
but silently drops every net that is only wire -- the old sheets labelled
every pin, so it never showed. Board A's generator is unchanged.

single.html: an SCH tab in the viewer (sch.js) -- the sheets as KiCad
plots them, a sheet list, drag to pan, scroll to zoom, a PDF of the lot.
tools/regen.py plots them into img/sch/s/ (--sch for that alone).

Co-Authored-By: Claude Opus 5.5 (1M context) <noreply@anthropic.com>
Connections:
- net +3V3A: no longer names the net of C716.1, R703.2, U7.44 (ADC_AVDD)
- net USB_DM_C: no longer names the net of R708.2, U7.51 (USB_DM)
- net USB_DP_C: no longer names the net of R707.2, U7.52 (USB_DP)
- net VREG_AVDD: no longer names the net of C718.1, R706.2, U7.46 (VREG_AVDD)
- net VREG_LX: no longer names the net of L701.2, U7.48 (VREG_LX)
- net XIN: no longer names the net of C709.1, U7.21 (XIN), Y1.1
- net XOUT: no longer names the net of R702.1, U7.22 (XOUT)
- net XTAL2: no longer names the net of C710.1, R702.2, Y1.3
Other:
- note added: "Decoupling"
- note added: "Notes"
- note added: "RP2350A"
- note added: "RP2350A as Raspberry Pi's minimal design (RP-006440): the core supply is the chip's own switching regulator, VREG_LX through L701 to +1V1, which VREG_FB senses and DVDD takes. VREG_AVDD is +3V3 through R706 and C718. One 100n at each IOVDD pin (C701-C706); C714 4u7 at VREG_VIN. ADC_AVDD is +3V3 filtered by R703 and C716 (+3V3A). BOOTSEL: SW1 on sheet 05 pulls QSPI_SS low through R701 at reset. Th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"
- note removed: "ADC supply"
- note removed: "CPU"
- note removed: "USB"
- note removed: "clock"
- note removed: "core rail"
- note removed: "decoupling"
- note removed: "power sources"
- note removed: "reset"
- moved on the sheet: C701, C702, C703, C704, C705, C706, C707, C709, C710, C711, C712, C713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
