File: hardware/single_board/04_power.kicad_sch (KiCad schematic)
At the start: 47 parts, among them J1 PHASE_A, J2 PHASE_B, J3 PHASE_C, J4 VBUS, J5 GND, Q1001 2N7002, U11 LMR38010SDDAR, U12 LMR38010SDDAR

Commit message: Board S: bus on an XT30, set back from the edge; SIT3088s tidied; re-routed
J4 is now the rp2350-motor-controller's XT30 (AMASS XT30PW-M, C431092,
pin 1 GND, pin 2 VMOT) in place of the two bus pads. At the rim its pegs
land on both RS-485 ports and no other rim takes a JST SH, so it sits 5 mm
back with the plug's path kept clear; its pins land at R 14.5.

- placement_s: bus="xt30" arrangement; the XT30 placed by its body with a
  peg rule; C1001 to 135 deg; SMDJ54A under the XT30; SM712 stacks; the four
  SIT3088 turned alike facing the ports (put_rigid, pair) with their escape
  strips kept clear; divider as one row; SPINE keepout
- gen_boards: project copy of the XT30 footprint with its courtyard round
  the part; In2 tab over the VMOT pin; spine from it to the header; In2
  no-via fences over the narrow VBUS fingers (a route cut C1007's)
- fanout.pin_field: via fields round the XT30 pins; finish.py honours via
  keepouts on any layer
- P5S re-run with the XT30's bus current: 0.009-0.016 deg alone
- routed: 1913 segments, 411 vias, 0 unconnected, DRC/ERC/netlist clean
- single.html: the XT30 section; "Where it is" below the viewer

Co-Authored-By: Claude Opus 5.5 (1M context) <noreply@anthropic.com>
Parts:
- removed J5: GND, servodrive:BusPad_Arc, symbol Connector:Conn_01x01_Pin
- J4: value VBUS -> XT30; footprint servodrive:BusPad_Arc -> servodrive:AMASS_XT30PW-M_1x02_P2.50mm_Horizontal; symbol Connector:Conn_01x01_Pin -> Connector_Generic:Conn_01x02
Connections:
- net GND: now also J4.1 (Pin_1)
- net VBUS: now also J4.2 (Pin_2); no longer J4.1 (Pin_1)
Other:
- note added: "bus: input"
- note removed: "bus input"
- moved on the sheet: C1001, C1002, C1003, C1004, C1005, C1006, C1007, C1008, C1009, C1010, C1011, C603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

Commit message: Board S schematic: drawn as a person would draw it, and on the page
The sheets were a grid of parts with a stub and a label on every pin.
tools/schdraw.py now draws a netlist from a hand-written layout: parts
placed and turned, wires between the pins that belong together, T-joins
split with a junction dot, ground and supply symbols on power pins, labels
only where a signal leaves its block. tools/schlayout_s.py is board S's
five sheets: signal left to right, supplies up, ground down, each part's
support parts at the pin they serve, dashed frames and notes. The header
pins and the notes follow the netlist, so a pin-map change redraws itself.

The drawing cannot change the circuit: every sheet is checked against
schematic_s's netlist before it is written, and `schdraw.py --check s`
compares KiCad's own netlist export net by net. It matches; ERC is 0 at
every severity; PCB parity is unchanged (the same 219 reports as before).

Found on the way: a symbol's instance path must be /<root>/<sheet>. With
the root left out, as schematic.py writes it, KiCad joins labelled nets
but silently drops every net that is only wire -- the old sheets labelled
every pin, so it never showed. Board A's generator is unchanged.

single.html: an SCH tab in the viewer (sch.js) -- the sheets as KiCad
plots them, a sheet list, drag to pan, scroll to zoom, a PDF of the lot.
tools/regen.py plots them into img/sch/s/ (--sch for that alone).

Co-Authored-By: Claude Opus 5.5 (1M context) <noreply@anthropic.com>
Connections:
- net +5V_BUCK: no longer names the net of C1010.1, C1011.1, C604.1, D1003.2 (A), L1002.2, R1006.1
- net BOOT_12V: no longer names the net of C1005.1, U11.7 (BOOT)
- net BOOT_5V: no longer names the net of C1008.1, U12.7 (BOOT)
- net EN_12V: no longer names the net of Q1001.3 (D), R1003.2, R1004.1, U11.2 (EN)
- net FB_12V: no longer names the net of R1001.2, R1002.1, U11.5 (FB)
- net FB_5V: no longer names the net of R1006.2, R1007.1, U12.5 (FB)
- net RT_12V: no longer names the net of R1008.1, U11.4 (RT/SYNC)
- net RT_5V: no longer names the net of R1009.1, U12.4 (RT/SYNC)
- net SW_12V: no longer names the net of C1005.2, L1001.1, U11.8 (SW)
- net SW_5V: no longer names the net of C1008.2, L1002.1, U12.8 (SW)
- net VDIV_MID: no longer names the net of R801.2, R806.1
Other:
- note added: "Bus input"
- note added: "Bus: 48 V operating on 80 V FETs. D1001 (SMDJ54A, 54 V standoff) clamps it; C1001 and C1002 are the bulk. VBUS_SENSE = VBUS x 4k7 / 116k7 (0.1 %), on ADC2. 12 V gate rail: LMR38010, starting at 9.9 V on the R1003/R1004 divider. GATE_OFF (GPIO14) high turns Q1001 on and stops the rail, taking the gate drivers' supply away. R1005 holds it low through reset, so the rail comes up and the drivers brak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"
- note added: "Mounting and motor leads"
- note added: "Notes"
- note removed: "bus voltage"
- note removed: "bus: TVS and bulk"
- note removed: "bus: input"
- note removed: "heatsink and mounting"
- note removed: "motor leads"
- note removed: "power sources"
- moved on the sheet: C1001, C1002, C1003, C1004, C1005, C1006, C1007, C1008, C1009, C1010, C1011, C603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
