File: hardware/single_board/05_io.kicad_sch (KiCad schematic)
At the start: 36 parts, among them J12 USB-C, J13 EXPANSION, J14 RS485 IN, J15 RS485 OUT, SW1 BOOTSEL, U13 USBLC6-2SC6, U14 SIT3088ETK, U15 SIT3088ETK, U17 SIT3088ETK, U18 SIT3088ETK

Commit message: Board S schematic: drawn as a person would draw it, and on the page
The sheets were a grid of parts with a stub and a label on every pin.
tools/schdraw.py now draws a netlist from a hand-written layout: parts
placed and turned, wires between the pins that belong together, T-joins
split with a junction dot, ground and supply symbols on power pins, labels
only where a signal leaves its block. tools/schlayout_s.py is board S's
five sheets: signal left to right, supplies up, ground down, each part's
support parts at the pin they serve, dashed frames and notes. The header
pins and the notes follow the netlist, so a pin-map change redraws itself.

The drawing cannot change the circuit: every sheet is checked against
schematic_s's netlist before it is written, and `schdraw.py --check s`
compares KiCad's own netlist export net by net. It matches; ERC is 0 at
every severity; PCB parity is unchanged (the same 219 reports as before).

Found on the way: a symbol's instance path must be /<root>/<sheet>. With
the root left out, as schematic.py writes it, KiCad joins labelled nets
but silently drops every net that is only wire -- the old sheets labelled
every pin, so it never showed. Board A's generator is unchanged.

single.html: an SCH tab in the viewer (sch.js) -- the sheets as KiCad
plots them, a sheet list, drag to pan, scroll to zoom, a PDF of the lot.
tools/regen.py plots them into img/sch/s/ (--sch for that alone).

Co-Authored-By: Claude Opus 5.5 (1M context) <noreply@anthropic.com>
Connections:
- net CC1: no longer names the net of J12.A5 (CC1), R1101.1
- net CC2: no longer names the net of J12.B5 (CC2), R1102.1
- net LED_B_K: no longer names the net of D1103.3 (BK), R1109.2
- net LED_G_K: no longer names the net of D1103.2 (GK), R1108.2
- net LED_R_K: no longer names the net of D1103.1 (RK), R1107.2
- net RS485_IN_DN_N: no longer names the net of D1101.2 (A2), J14.3 (Pin_3), R1105.2, U14.7 (B)
- net RS485_IN_DN_P: no longer names the net of D1101.1 (A1), J14.2 (Pin_2), R1105.1, U14.6 (A)
- net RS485_IN_UP_N: no longer names the net of D1102.2 (A2), J14.5 (Pin_5), U15.7 (B)
- net RS485_IN_UP_P: no longer names the net of D1102.1 (A1), J14.4 (Pin_4), U15.6 (A)
- net RS485_OUT_DN_N: no longer names the net of D1104.2 (A2), J15.3 (Pin_3), U17.7 (B)
- net RS485_OUT_DN_P: no longer names the net of D1104.1 (A1), J15.2 (Pin_2), U17.6 (A)
- net RS485_OUT_UP_N: no longer names the net of D1105.2 (A2), J15.5 (Pin_5), R1106.2, U18.7 (B)
- net RS485_OUT_UP_P: no longer names the net of D1105.1 (A1), J15.4 (Pin_4), R1106.1, U18.6 (A)
Other:
- note added: "ADC3 divider, FAULT_n pull-up"
- note added: "Expansion header: PD or Ethernet board"
- note added: "RS-485 is a CPU relay: each port is two point- to-point pairs, one in and one out, so a drive passes the chain on in software. Drivers are always enabled; each receiver has its 120R termination (R1105, R1106). R803 with the NTC (R901, sheet 01) makes FET_TEMP."
- note added: "RS-485 relay: port IN"
- note added: "RS-485 relay: port OUT"
- note added: "Status LED, BOOTSEL, test pads"
- note removed: "ADC3 front end, FAULT_n"
- note removed: "RS-485 relay"
- note removed: "expansion header: PD or Ethernet board"
- note removed: "status LED, BOOTSEL, test pads"
- moved on the sheet: C1102, C1103, C1104, C1105, C802, D1002, D1101, D1102, D1103, D1104, D1105, J12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
