File: hardware/single_board/02_power.kicad_sch (KiCad schematic)
At the start: 46 parts, among them J1 PHASE_A, J2 PHASE_B, J3 PHASE_C, J4 XT30, Q1001 2N7002, U11 LMR38010SDDAR, U12 LMR38010SDDAR

Commit message: Board S schematic on three sheets: bridge + CPU, power, encoder + IO
Asked for fewer pages: the power bridge goes with the CPU that drives it
(A2), the encoder with the rest of the IO (A3); the supplies keep their
sheet. schematic_s.SHEET_OF maps the parts' sheet names (board A keeps its
own), and schdraw.Sheet.origin() lets a sheet place layouts written in their
own coordinates side by side. HIN/LIN and the other CPU-to-bridge nets are
now local labels on one sheet. The notes say which sheet a part is on.

KiCad's netlist matches schematic_s.nets(); ERC 0. The board is linked to
the netlist by reference, so the PCB is untouched.

Co-Authored-By: Claude Opus 5.5 (1M context) <noreply@anthropic.com>
Other:
- title: servodrive — board S, single board — 04_power -> servodrive — board S, single board — 02_power

Commit message: Board S with six D6.3 bulk cans: routed, DRC 0; the bulk options page
The two D10 cans carried 6.4 A of ripple each at 20 A RMS per phase, 3.7
times their rating at 20-40 kHz. Six PA100V22M6X9 (22 uF, 2.6 A) carry
2.3 A each, within rating to 16 A per phase continuously, 0.15 W a can.

Routed with the maze making the RS-485 IN pair and the encoder's CS and DO
before the router, then targeted rip-ups for EXP_GP24, HIN_A and SWCLK.
2241 segments, 444 vias; DRC 0 all severities, ERC 0, parity 219 of the
same kinds as before, netlist diff and deadcheck clean. bulk.html has the
parts, the banks through the DC-link network, what fits and what routed.
ethernet.html: the can holes, and GPIO14 is port OUT's UART now.

Co-Authored-By: Claude Opus 5.5 (1M context) <noreply@anthropic.com>
Parts:
- added C1012, C1013, C1014, C1015: 22u/100V polymer, Capacitor_THT:CP_Radial_D6.3mm_P2.50mm, symbol Device:C_Polarized
- C1001, C1002: value 100u/100V polymer -> 22u/100V polymer; footprint Capacitor_THT:CP_Radial_D10.0mm_P5.00mm -> Capacitor_THT:CP_Radial_D6.3mm_P2.50mm
Connections:
- net GND: now also C1012.2, C1013.2, C1014.2, C1015.2
- net VBUS: now also C1012.1, C1013.1, C1014.1, C1015.1
Other:
- note added: "Bus: 48 V operating on 80 V FETs. D1001 (SMDJ54A, 54 V standoff) clamps it; C1001, C1012, C1002, C1015, C1013 and C1014 are the bulk. VBUS_SENSE = VBUS x 4k7 / 116k7 (0.1 %), on ADC2. 12 V gate rail: LMR38010, starting at 9.9 V on the R1003/R1004 divider. GATE_OFF (GPIO2) high turns Q1001 on and stops the rail, taking the gate drivers' supply away. R1005 holds it low through reset, so the rail co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"
- note removed: "Bus: 48 V operating on 80 V FETs. D1001 (SMDJ54A, 54 V standoff) clamps it; C1001 and C1002 are the bulk. VBUS_SENSE = VBUS x 4k7 / 116k7 (0.1 %), on ADC2. 12 V gate rail: LMR38010, starting at 9.9 V on the R1003/R1004 divider. GATE_OFF (GPIO14) high turns Q1001 on and stops the rail, taking the gate drivers' supply away. R1005 holds it low through reset, so the rail comes up and the drivers brak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"
- moved on the sheet: C1002, C801, R801, R802, R806
