File: hardware/single_board/01_bridge_cpu.kicad_sch (KiCad schematic)
At the start: 106 parts, among them Q1 BSC030N08NS5, Q2 BSC030N08NS5, Q3 BSC030N08NS5, Q4 BSC030N08NS5, Q5 BSC030N08NS5, Q6 BSC030N08NS5, U1 EG2103, U2 EG2103, U3 EG2103, U4 INA241A3, U5 INA241A3, U6 INA241A3, U7 RP2350A, U8 W25Q16JVUXIQ, U9 SPX3819M5-3.3, Y1 12MHz

Commit message: Board S: SIT65HVD75ETK and W25Q80DVUXIE for the parts that went out of stock
Every placed part re-checked at JLCPCB on 2026-10-16: the SIT3088ETK and
the W25Q16JVUXIQ were at zero. The SIT65HVD75ETK is the same MAX3485
pinout in the same DFN-8 3x3 (C7433976, 20,671 in stock), and its receiver
threshold (V_IT+ <= -10 mV) reads a terminated idle pair as a 1, which
answers the fail-safe item on paper. The W25Q80DVUXIE is the same pins and
USON 2x3 land pattern, 8 Mbit (C401667, 8,611): firmware needs
PICO_FLASH_SIZE_BYTES 1 MB and has to set QE, which it ships clear.

Board S only (schematic_s overrides; board A keeps the W25Q16JV): two new
derived symbols appended to the library, the two sheets regenerated, the
routed board's value fields patched, the fan-out's escape rule taking the
new name. ERC 0, netlist == schematic_s, DRC 0 / 0 unconnected, schematic
parity the same 219 items as before. Viewer rebuilt.

Still short: the RP2350's 3.3 uH AOTA-B201610S3R3 (9) and TPSMF4L54A (42,
three a board).

Co-Authored-By: Claude Opus 5.5 <noreply@anthropic.com>
Parts:
- U8: value W25Q16JVUXIQ -> W25Q80DVUXIE; symbol servodrive:W25Q16JV -> servodrive:W25Q80DV
Changed lines of the file:
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@@
 	)
 	(symbol
-		(lib_id "servodrive:W25Q16JV")
+		(lib_id "servodrive:W25Q80DV")
 		(at 271.7800 135.8900 0)
 		(unit 1)
@@
 			(at 283.2100 142.2400 0)
 			(effects (font (size 1.27 1.27)) (justify left)))
-		(property "Value" "W25Q16JVUXIQ"
+		(property "Value" "W25Q80DVUXIE"
 			(at 283.2100 144.7800 0)
 			(effects (font (size 1.27 1.27)) (justify left)))
